Commit message: Refactor Mowgli packages and improve simulation environment
- Updated package.xml to replace rosbridge_server and rosapi with foxglove_bridge for GUI integration.
- Removed Gazebo plugins from mowgli.urdf.xacro, indicating that simulation physics and sensors are now defined in a separate Ignition Gazebo model.
- Added min_turning_radius parameter to coverage_planner.yaml for improved path planning.
- Removed unused datum parameters in gps_pose_converter_node.hpp and corresponding declarations in gps_pose_converter_node.cpp.
- Adjusted covariance values in wheel_odometry_node.cpp to reflect untrusted EKF usage.
- Reduced oscillation recovery thresholds in ftc_controller.hpp for better control responsiveness.
- Enhanced FTCController to find the nearest path point to the robot's position, improving path following accuracy.
- Increased wall height in empty_garden.sdf and garden.sdf to ensure LiDAR compatibility.
- Introduced precision_monitor.py for real-time precision metrics publishing to Foxglove, enhancing localization quality assessment.
- Updated mowgli.service to reflect the change from ROS 2 Humble to Jazzy.

File: src/mowgli_bringup/urdf/mowgli.urdf.xacro (robot description, xacro)
@@ -319,94 +319,8 @@
   </joint>
   <!-- ================================================================
-       Gazebo plugins
-       ================================================================ -->
-  <!-- Differential drive controller -->
-  <gazebo>
-    <plugin name="diff_drive" filename="libgazebo_ros_diff_drive.so">
-      <ros>
-        <namespace></namespace>
-      </ros>
-      <left_joint>left_wheel_joint</left_joint>
-      <right_joint>right_wheel_joint</right_joint>
-      <wheel_separation>${wheel_track}</wheel_separation>
-      <wheel_diameter>${2 * wheel_radius}</wheel_diameter>
-      <max_wheel_torque>20.0</max_wheel_torque>
-      <max_wheel_acceleration>2.0</max_wheel_acceleration>
-      <command_topic>cmd_vel</command_topic>
-      <odometry_topic>wheel_odom</odometry_topic>
-      <odometry_frame>odom</odometry_frame>
-      <robot_base_frame>base_footprint</robot_base_frame>
-      <publish_odom>true</publish_odom>
-      <publish_odom_tf>false</publish_odom_tf>
-      <publish_wheel_tf>false</publish_wheel_tf>
-      <update_rate>50.0</update_rate>
-    </plugin>
-  </gazebo>
-  <!-- IMU sensor -->
-  <gazebo reference="imu_link">
-    <sensor name="imu_sensor" type="imu">
-      <always_on>true</always_on>
-      <update_rate>100</update_rate>
-      <visualize>false</visualize>
-      <imu>
-        <angular_velocity>
-          <x><noise type="gaussian"><mean>0.0</mean><stddev>0.009</stddev></noise></x>
-          <y><noise type="gaussian"><mean>0.0</mean><stddev>0.009</stddev></noise></y>
-          <z><noise type="gaussian"><mean>0.0</mean><stddev>0.009</stddev></noise></z>
-        </angular_velocity>
-        <linear_acceleration>
-          <x><noise type="gaussian"><mean>0.0</mean><stddev>0.021</stddev></noise></x>
-          <y><noise type="gaussian"><mean>0.0</mean><stddev>0.021</stddev></noise></y>
-          <z><noise type="gaussian"><mean>0.0</mean><stddev>0.021</stddev></noise></z>
-        </linear_acceleration>
-      </imu>
-      <plugin name="imu_plugin" filename="libgazebo_ros_imu_sensor.so">
-        <ros>
-          <namespace></namespace>
-          <remapping>~/out:=imu/data</remapping>
-        </ros>
-        <initial_orientation_as_reference>false</initial_orientation_as_reference>
-      </plugin>
-    </sensor>
-  </gazebo>
-  <!-- 2-D LiDAR sensor (360 deg, 8 m range) -->
-  <gazebo reference="lidar_link">
-    <sensor name="lidar_sensor" type="ray">
-      <always_on>true</always_on>
-      <update_rate>10</update_rate>
-      <visualize>false</visualize>
-      <ray>
-        <scan>
-          <horizontal>
-            <samples>360</samples>
-            <resolution>1</resolution>
-            <min_angle>-3.14159</min_angle>
-            <max_angle>3.14159</max_angle>
-          </horizontal>
-        </scan>
-        <range>
-          <min>0.10</min>
-          <max>8.0</max>
-          <resolution>0.01</resolution>
-        </range>
-        <noise>
-          <type>gaussian</type>
-          <mean>0.0</mean>
-          <stddev>0.01</stddev>
-        </noise>
-      </ray>
-      <plugin name="lidar_plugin" filename="libgazebo_ros_ray_sensor.so">
-        <ros>
-          <namespace></namespace>
-          <remapping>~/out:=scan</remapping>
-        </ros>
-        <output_type>sensor_msgs/LaserScan</output_type>
-        <frame_name>lidar_link</frame_name>
-      </plugin>
-    </sensor>
-  </gazebo>
-  <!-- Base link colour in Gazebo -->
-  <gazebo reference="base_link">
-    <material>Gazebo/Green</material>
-  </gazebo>
+       Gazebo simulation
+       ================================================================ -->
+  <!-- Simulation physics and sensors are defined in the standalone Ignition
+       Gazebo model: mowgli_simulation/models/mowgli_mower/model.sdf
+       This URDF provides TF frames and RViz visualisation only. -->
 </robot>
