Commit message: fix: sync ros2/ with mowgli-ros2 main branch (#37)
* fix: sync gui/ with openmower-gui v3 branch

The monorepo imported gui/ from the topic-rename branch instead of v3,
missing 11 commits (robot footprint, dock visualization, chassis
dimensions, sensor positions, topic name fixes) and including an
unmerged topic-rename commit. This syncs gui/ to the v3 branch state,
reverting the /mowgli/ namespace changes in favor of the correct
/hardware_bridge/ remappings.

* fix: sync ros2/ with mowgli-ros2 main branch (hardware-tested)

The monorepo imported ros2/ from the topics-rename branch instead of
main, missing 42 commits with critical hardware fixes (opennav_docking,
GPS heading calibration, battery safety, SLAM reset, dock anchoring,
coverage checkpoint persistence) and including 20 topic-rename commits
that were never merged to main.

This syncs ros2/ to the mowgli-ros2 main branch state while preserving
monorepo-only additions:
- ExecuteFullCoveragePath BT node (replaces ExecuteSwathBySwath)
- use_lidar launch argument for GPS-only simulation
- xvfb headless rendering in Dockerfile
- Topic relay nodes for simulation

* chore: auto-format C++ files

* fix: update hardware bridge topic names and remove unused dependencies

* chore: auto-format C++ files

* fix: améliorer la gestion des processus ROS2 et la récupération en ligne dans les nœuds de comportement

* chore: auto-format C++ files

* Update copyright information and licensing details across the project files

- Updated copyright year to 2026 for all relevant source files, launch files, and test files.
- Changed licensing comments to reflect the GNU General Public License version 3, ensuring compliance and clarity regarding redistribution and modification rights.
- Ensured consistent formatting and style across all modified files to enhance readability and maintainability.

* fix: mettre à jour le modèle Claude et ajouter le jeton OAuth pour les actions de code

File: ros2/src/mowgli_bringup/urdf/mowgli.urdf.xacro (robot description, xacro)
@@ -20,38 +20,49 @@
        Configurable arguments (can be overridden via xacro command-line)
        ================================================================ -->
-  <xacro:arg name="lidar_x"   default="0.20"/>
+  <xacro:arg name="lidar_x"   default="0.38"/>
   <xacro:arg name="lidar_y"   default="0.0"/>
   <xacro:arg name="lidar_z"   default="0.22"/>
   <xacro:arg name="lidar_yaw" default="0.0"/>
-  <xacro:arg name="imu_x"     default="0.0"/>
+  <xacro:arg name="imu_x"     default="0.18"/>
   <xacro:arg name="imu_y"     default="0.0"/>
   <xacro:arg name="imu_z"     default="0.095"/>
   <xacro:arg name="imu_yaw"   default="0.0"/>
-  <xacro:arg name="gps_x"     default="0.0"/>
+  <xacro:arg name="gps_x"     default="0.3"/>
   <xacro:arg name="gps_y"     default="0.0"/>
   <xacro:arg name="gps_z"     default="0.20"/>
-  <!-- ================================================================
-       Properties
-       ================================================================ -->
-  <xacro:property name="base_length"     value="0.54"/>
-  <xacro:property name="base_width"      value="0.40"/>
-  <xacro:property name="base_height"     value="0.19"/>
-  <!-- Rear drive wheels (from real URDF: diameter 0.0895m) -->
-  <xacro:property name="wheel_radius"    value="0.04475"/>
-  <xacro:property name="wheel_width"     value="0.04"/>
-  <xacro:property name="wheel_track"     value="0.40"/>  <!-- centre-to-centre -->
-  <xacro:property name="wheel_mass"      value="0.5"/>
-  <!-- Rear wheels are offset behind base_link centre -->
-  <xacro:property name="wheel_x_offset"  value="-0.18"/>
-  <!-- Front caster wheels (smaller) -->
-  <xacro:property name="caster_radius"   value="0.03"/>
-  <xacro:property name="caster_width"    value="0.03"/>
-  <xacro:property name="caster_mass"     value="0.2"/>
-  <xacro:property name="caster_x_offset" value="0.22"/>
-  <xacro:property name="caster_track"    value="0.36"/>  <!-- centre-to-centre -->
-  <xacro:property name="base_mass"       value="8.76"/>
-  <xacro:property name="blade_radius"    value="0.09"/>
-  <xacro:property name="blade_height"    value="0.01"/>
-  <xacro:property name="blade_mass"      value="0.3"/>
+  <!-- Chassis shape (all from mowgli_robot.yaml via launch file) -->
+  <xacro:arg name="chassis_length"   default="0.54"/>
+  <xacro:arg name="chassis_width"    default="0.40"/>
+  <xacro:arg name="chassis_height"   default="0.19"/>
+  <xacro:arg name="chassis_center_x" default="0.18"/>
+  <xacro:arg name="wheel_radius"     default="0.04475"/>
+  <xacro:arg name="wheel_width"      default="0.04"/>
+  <xacro:arg name="wheel_track"      default="0.325"/>
+  <xacro:arg name="wheel_x_offset"   default="0.0"/>
+  <xacro:arg name="caster_radius"    default="0.03"/>
+  <xacro:arg name="caster_track"     default="0.36"/>
+  <xacro:arg name="blade_radius"     default="0.09"/>
+  <!-- ================================================================
+       Properties (resolved from args — all shape from config)
+       ================================================================ -->
+  <xacro:property name="base_length"      value="$(arg chassis_length)"/>
+  <xacro:property name="base_width"       value="$(arg chassis_width)"/>
+  <xacro:property name="base_height"      value="$(arg chassis_height)"/>
+  <xacro:property name="chassis_cx"       value="$(arg chassis_center_x)"/>
+  <xacro:property name="wheel_radius"     value="$(arg wheel_radius)"/>
+  <xacro:property name="wheel_width"      value="$(arg wheel_width)"/>
+  <xacro:property name="wheel_track"      value="$(arg wheel_track)"/>
+  <xacro:property name="wheel_mass"       value="0.5"/>
+  <xacro:property name="wheel_x_offset"   value="$(arg wheel_x_offset)"/>
+  <xacro:property name="caster_radius"    value="$(arg caster_radius)"/>
+  <xacro:property name="caster_width"     value="0.03"/>
+  <xacro:property name="caster_mass"      value="0.2"/>
+  <!-- Casters near front edge of chassis -->
+  <xacro:property name="caster_x_offset"  value="${chassis_cx + base_length/2.0 - caster_radius}"/>
+  <xacro:property name="caster_track"     value="$(arg caster_track)"/>
+  <xacro:property name="base_mass"        value="8.76"/>
+  <xacro:property name="blade_radius"     value="$(arg blade_radius)"/>
+  <xacro:property name="blade_height"     value="0.01"/>
+  <xacro:property name="blade_mass"       value="0.3"/>
   <!-- Derived: base_link is wheel_radius above ground -->
   <xacro:property name="base_z_offset"   value="${wheel_radius}"/>
@@ -106,9 +117,10 @@
   </joint>
   <!-- ================================================================
-       base_link  (geometric centre of chassis at wheel axle height)
+       base_link  (centre of rear drive wheel axis at wheel axle height)
        ================================================================ -->
   <link name="base_link">
     <visual>
-      <origin xyz="0 0 ${base_height/2}" rpy="0 0 0"/>
+      <!-- Chassis centre offset forward from wheel axis -->
+      <origin xyz="${chassis_cx} 0 ${base_height/2}" rpy="0 0 0"/>
       <geometry>
         <box size="${base_length} ${base_width} ${base_height}"/>
@@ -119,5 +131,5 @@
     </visual>
     <collision>
-      <origin xyz="0 0 ${base_height/2}" rpy="0 0 0"/>
+      <origin xyz="${chassis_cx} 0 ${base_height/2}" rpy="0 0 0"/>
       <geometry>
         <box size="${base_length} ${base_width} ${base_height}"/>
@@ -156,5 +168,5 @@
       <parent link="base_link"/>
       <child  link="${side}_wheel_link"/>
-      <!-- Rear drive wheels: offset behind base_link centre -->
+      <!-- Drive wheels at base_link origin -->
       <origin xyz="${wheel_x_offset} ${y_reflect * wheel_track/2} 0" rpy="0 0 0"/>
       <axis xyz="0 1 0"/>
@@ -242,6 +254,6 @@
     <parent link="base_link"/>
     <child  link="blade_link"/>
-    <!-- Blade disc centred under base, matching real robot -->
-    <origin xyz="0 0 ${-wheel_radius + 0.05}" rpy="0 0 0"/>
+    <!-- Blade disc centred under chassis -->
+    <origin xyz="${chassis_cx} 0 ${-wheel_radius + 0.05}" rpy="0 0 0"/>
     <axis xyz="0 0 1"/>
   </joint>
