Commit message: fix(sim): make Webots Phase 1 controller-manager-ready
The Phase 1 scaffold booted Webots and brought up the IPC bridge,
but the WebotsController crashed shortly after with
`terminate called: Joint 'left_wheel_motor' not found in URDF`
followed by a segfault — the joint-limits code path in
hardware_interface (kilted+) requires every <ros2_control> joint to
also exist as a real <joint> element in the URDF so it can read
limits, and the scaffold URDF only declared a single base_link.

Three coordinated fixes get cmd_vel → /wheel_odom_raw working with
ω measured to 0.7999 rad/s for a commanded 0.8 rad/s (steady state,
< 0.01 % error):

* urdf_webots/mowgli_webots.urdf — flesh out the kinematic tree
  (base_link, base_footprint, left_wheel, right_wheel, lidar_link,
  imu_link, gps_link) with proper <link>/<joint> blocks. Wheels
  are continuous joints around Y with the same anchors as the
  inline Robot {} in mowgli_garden.wbt (axis 0 1 0,
  origin xyz="0 ±0.1625 -0.10"), and carry effort/velocity limits
  matching the .wbt RotationalMotor caps. Inertials are deliberately
  left off chassis + wheels — Webots owns the physics, and KDL
  warns when the URDF root link has an inertia.

* launch/webots_minimal.launch.py — three independent hardenings:
  - respawn=False on the WebotsController (a respawn loop produced
    "ExecuteLocal action 'spawner-7': executed more than once" and
    masked the underlying crash).
  - controller-manager-timeout 50 → 90 s (Xvfb boot + IPC handshake
    + URDF parse + hardware-interface init has more headroom now).
  - set_robot_state_publisher: True → False (we already run our
    own RSP with the same URDF; the driver's republish would race
    on the transient_local /robot_description latch).

* worlds_webots/mowgli_garden.wbt — basicTimeStep 16 → 20 ms so
  the Webots physics step matches the controller_manager 50 Hz
  update_rate exactly (Webots warns otherwise).

Verified end-to-end:
  ros2 launch mowgli_simulation webots_minimal.launch.py mode:=fast
  ros2 topic pub --rate 20 /cmd_vel geometry_msgs/msg/TwistStamped \\
    '{twist: {linear: {x: 0.0}, angular: {z: 0.8}}}'
  ros2 topic echo /wheel_odom_raw --field twist.twist.angular.z
  → steady-state 0.7999 rad/s (commanded 0.8). Linear 0.2 m/s
  command also tracks within wheel-slip tolerance.

File: ros2/src/mowgli_simulation/urdf_webots/mowgli_webots.urdf (robot description, URDF)
Before this commit: robot MowgliMower, 1 links, 0 joints
Links:
- added link base_footprint
- added link gps_link
- added link imu_link
- added link left_wheel; collision cylinder length=0.04 radius=0.093; visual cylinder length=0.04 radius=0.093
- added link lidar_link
- added link right_wheel; collision cylinder length=0.04 radius=0.093; visual cylinder length=0.04 radius=0.093
- link base_link: geometry collision box size=0.60 0.40 0.19; visual box size=0.60 0.40 0.19
Joints:
- added joint base_link_to_base_footprint: type fixed, parent base_link, child base_footprint, origin xyz=0 0 -0.10 rpy=0 0 0
- added joint base_link_to_gps: type fixed, parent base_link, child gps_link, origin xyz=0.30 0 0.10 rpy=0 0 0
- added joint base_link_to_imu: type fixed, parent base_link, child imu_link, origin xyz=0 0 0 rpy=0 0 0
- added joint base_link_to_lidar: type fixed, parent base_link, child lidar_link, origin xyz=0 0.024 0.12 rpy=0 0 3.1408
- added joint left_wheel_motor: type continuous, parent base_link, child left_wheel, origin xyz=0 0.1625 -0.10 rpy=0 0 0, axis 0 1 0, limit effort=10.0 velocity=100.0
- added joint right_wheel_motor: type continuous, parent base_link, child right_wheel, origin xyz=0 -0.1625 -0.10 rpy=0 0 0, axis 0 1 0, limit effort=10.0 velocity=100.0
