Commit message: fix(sim): Webots Phase 2 partial — TF chain + IMU topic wiring
Two coordinated fixes that get the full Mowgli stack booting cleanly on
Webots and the BT advancing through MOWING; the BackUp/cmd_vel motion
itself is still blocked by a chassis-tip pathology in the inline robot
(see Blocker section below).

* ros2/src/mowgli_simulation/urdf_webots/mowgli_webots.urdf
    Invert the base_link↔base_footprint joint so base_footprint is the
    PARENT (REP-105). Phase 1 worked with the wrong direction because no
    ekf_odom was running; Phase 2 brings up ekf_odom_node which publishes
    odom→base_footprint, so RSP also publishing base_link→base_footprint
    gave base_footprint two parents and tf2 silently picked the wrong
    chain — Nav2 lookups against a stale TF, cmd_vel never reaching the
    diff_drive_controller in the right frame.
    Wheel anchor stays at z=-0.10 (matching the .wbt's intentionally
    half-buried cylinders); annotated to make the geometric contract
    explicit and survive future refactors.

* ros2/src/mowgli_bringup/launch/sim_full_system.launch.py
    Two changes:
    - Pass mode:=fast through to webots_minimal.launch.py so the BT
      can actually progress through Nav2 lifecycle activation, RecordArea,
      MOWING etc. within reasonable wall-clock time (Webots default
      "realtime" mode otherwise tops out at ~1×).
    - Fix sim_imu_noise input_topic from /imu/data_raw (Gazebo-era
      name) to /imu/data_sim (what the Webots Ros2IMU plugin actually
      publishes per mowgli_webots.urdf). Without this, robot_localization
      saw zero IMU input, ekf_map_node never converged, and the
      wait_for_map_odom_tf gate never released → Nav2 lifecycle stayed
      down forever.

Tested
------
With these two changes:
  * sim_full_system.launch.py boots cleanly under DISPLAY=:99 and Webots
    fast mode. All Nav2 lifecycle nodes activate (controller_server,
    planner_server, behavior_server, bt_navigator, waypoint_follower,
    docking_server, collision_monitor).
  * map → odom TF resolves within ~1.5 s of bringup.
  * BT loads main_tree.xml, reaches IDLE_DOCKED, accepts COMMAND_START
    via /behavior_tree_node/high_level_control once SetNavMode finishes
    waiting for controller_server params.
  * BT advances PREFLIGHT_CHECK → UNDOCKING → BackUp action dispatched
    to behavior_server with the correct 1 m / 0.20 m/s payload.

Blocker (unresolved, documented for next session)
-------------------------------------------------
The inline Mowgli robot in worlds_webots/mowgli_garden.wbt has a
chassis-tip pathology that prevents real translation under cmd_vel.
The wheels rotate correctly (Phase 1 verified ω_cmd vs ω_measured at
<0.01 % error), but the chassis itself either:
  (a) tips forward 30–45° within 5 s of any 0.2 m/s cmd_vel and ends
      up rolling on its nose (with the casters lifted to anchor z=-0.07
      so they "just touch"), OR
  (b) translates only 2-3 cm out of 1 m commanded with the original
      half-buried casters (z=-0.13) — wheels spin against the floor
      with ~95 % slip because the contact-point shift in ODE eats the
      rotation.

Things tried in this session and reverted:
  - Lift wheel anchor to z=-0.007 (just touch the floor): casters lift
    under acceleration, robot somersaults forward.
  - Lower CoM to robot z=-0.10 (= world z=0): no effect on the tip.
  - Cap motor maxTorque to 2 Nm and add 4 rad/s² acceleration limit:
    chassis still tips, just more slowly.
  - Shrink chassis bounding box to a thin slab above the wheels: no
    effect.
  - High coulombFriction (5.0) + larger softCFM: no effect on slip.
  - Various combinations of the above + Robot world z lift (0.193) +
    matching caster anchor (-0.163): same outcomes.

Likely root cause is a combination of:
  - Sphere casters on BallJoints with no rolling-resistance modelling
    in Webots ODE — once the casters lift, nothing damps the tip.
  - The chassis Robot.boundingObject Box overlapping with wheel and
    caster Solids, even with self-collision disabled — the contact
    solver appears to fight the joint constraints in a way that
    bleeds energy out of translation.
  - Static stability is fine (robot rests level at IMU pitch ≈ 0°);
    the failure is dynamic, triggered by motor torque reaction +
    longitudinal weight transfer when the diff_drive_controller's
    velocity-control PID slams the wheels from 0 to commanded ω in
    one timestep.

Next steps for the next session:
  - Replace the inline Robot{} with one of the Webots PROTOs from
    webots_ros2_husarion (rosbot, rosbot_xl) and remap the joint
    names — the PROTO models are tuned for stable diff-drive motion
    and ship with the right friction/inertia parameters out of the box.
  - Or rewrite the inline robot using the design pattern from a
    Webots-shipped 4-wheel mower example (if one exists), keeping the
    Mowgli sensor mounts but borrowing the chassis + wheel + caster
    physics block verbatim.
  - The BT/Nav2 plumbing on top is now correct and will pick up the
    new robot transparently once cmd_vel actually translates.

Other observations worth flagging (not Webots bugs, but exercised
differently in sim than on real hardware):
  - costmap_scan_filter prints "ground filter idle: last IMU sample
    Ns old" warnings that are harmless when IMU pitch is small but
    spam the log when the robot tips. Threshold is in seconds and
    the warning text uses sim time delta from the last IMU stamp,
    which becomes huge once the IMU subscriber is starved.
  - opennav_docking warns "Parameter dock_backwards is deprecated"
    on every boot — pre-existing, not Webots-related.
  - SetNavMode hits a 20 s wall while controller_server is loading,
    which the BT should already tolerate (RetryUntilSuccessful around
    the GPSModeSelector branch), but COMMAND_START sent BEFORE the
    first successful SetNavMode silently fails the GPS mode selector
    and the IDLE branch holds. Resending COMMAND_START after
    "SetNavMode: mode set to 'precise'" appears in the log advances
    the BT correctly. Worth adding a smaller/faster fallback timeout
    in SetNavMode itself.

File: ros2/src/mowgli_simulation/urdf_webots/mowgli_webots.urdf (robot description, URDF)
Before this commit: robot MowgliMower, 7 links, 6 joints
Joints:
- removed joint base_link_to_base_footprint
- added joint base_footprint_to_base_link: type fixed, parent base_footprint, child base_link, origin xyz=0 0 0.10 rpy=0 0 0
